File: sfp_v4.sch (KiCad schematic (older format))
At the start: 75 parts, among them J102 SMA, J104 SMA, J106 SMA, P101 SFP-CONNECTOR, P103 CONN_01X01, P106 CONN_01X01, T101 ADT2-1T, T102 ADT2-1T, U101 LMH6702, U102 LMH6702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

Commit message: adjust values
Parts:
- R119, R133: value 150R -> 0R
Changed lines of the file:
@@
 P 5050 1700
 F 0 "R119" V 5130 1700 50  0000 C CNN
-F 1 "150R" V 5050 1700 50  0000 C CNN
+F 1 "0R" V 5050 1700 50  0000 C CNN
 F 2 "Resistors_SMD:R_0805" V 4980 1700 30  0001 C CNN
 F 3 "" H 5050 1700 30  0000 C CNN
@@
 P 7850 2950
 F 0 "R133" V 7930 2950 50  0000 C CNN
-F 1 "150R" V 7850 2950 50  0000 C CNN
+F 1 "0R" V 7850 2950 50  0000 C CNN
 F 2 "Resistors_SMD:R_0805" V 7780 2950 30  0001 C CNN
 F 3 "" H 7850 2950 30  0000 C CNN
